File: hardware/v1/sequencer.kicad_pcb (KiCad board)
At the start: 2 copper layers, 102.2 x 73.7 mm, 115 parts, among them J1 CV A OUT, J10 power_panel, J11 keys_board, J12 keys_panel, J13 CLOCK_OUT, J14 GATE A, J15 GATE B, J16 leds_board, J17 leds_wire, J18 CLK IN, J19 panel, J2 seq_a_board, J20 CLK RATE, J21 panel, J22 CLK OUT, J23 panel, J24 GATE A, J25 panel, J26 GATE B, J27 panel, J28 SEQ MODE, J29 panel, J3 seq_a_panel, J30 STEP CNT, J31 panel, J32 GATE PGM, J33 gate_pgm_panel, J34 RESET, J35 panel, J36 RST SW, J37 panel, J38 power_board_input, J39 STEP CNT SW, J4 CV B OUT, J40 panel, J5 RESET_IN, J6 seq_b_board, J7 seq_b_panel, J8 CLOCK_IN, J9 power_board, SW1 SW_DPDT_x2, SW10 SW_Push, SW11 SW_Push, SW12 SW_Push, SW2 SW_SPDT_MSM, SW3 SW_SPST, SW4 SW_SPDT_MSM, SW5 SW_Push, SW6 SW_Push, SW7 SW_Push, SW8 SW_Push, SW9 SW_Push, U1 74HC595, U2 74HC595, U3 4051

Commit message: Added readme
Parts:
- removed D21, D27: LED, LED_THT:LED_D5.0mm
- R10: value 100k -> 10k
Routing:
- net GNDA: track 1123.4 -> 1113.5 mm
- net Net-(J19-Pad1): track 11.4 -> 5.08 mm
